File: Circuit/IRis - Slave PCB Layout (CR2032).brd (EAGLE design)
At the start: 30.5 x 59.7 mm, 19 parts

Commit message: PCB Layout Included For AA Cell and CR2032 Cell. Gerber Files Added
Parts:
- removed E$17, E$18: (no value), wirepad:1,6/0,8
- removed E$19: (no value), holes:2,8
- E$16: device SparkFun-Switches:SWITCH_SPDT_PTH_11.6X4.0MM -> SparkFun-Batteries:BATTCOM_20MM_PTH
- moved E$11 12.5 mm to (24.1, 17.8), turned to 270 degrees
- moved E$9 10.2 mm to (21.6, 22.9)
- moved E$16 6.84 mm to (11.4, 12.7), turned to 315 degrees
- moved E$8 5.24 mm to (24.1, 27.9)
- moved E$10 1.27 mm to (21.6, 33.0), turned to 270 degrees
Connections:
- removed net S$12: E$16.3, E$17.1
- net GND: now also E$5.4; no longer E$16.1
- net S$1: now also E$10.P$2; no longer E$10.P$1
- net S$2: now also E$1.5, E$1.8, E$10.P$1, E$13.P$2, E$16.1, E$6.VCC; no longer E$3.4, E$8.P$1, E$9.P$2
- net S$3: now also E$3.4, E$8.P$1, E$9.P$2; no longer E$11.P$1, E$4.4, E$9.P$1
- net S$6: now also E$11.P$1, E$4.4, E$9.P$1; no longer E$1.5, E$1.8, E$10.P$2, E$13.P$2, E$18.1, E$6.VCC
Routing:
- net S$6: track 75.6 -> 7.63 mm
- net S$2: track 9.71 -> 68.1 mm
- net GND: track 81.2 -> 93.1 mm
- net S$12: track 8.98 -> 0.00 mm
- net S$3: track 12.2 -> 7.63 mm
- net S$1: track 5.54 -> 7.86 mm
Other:
- board text added: "1"
- board text added: "100k"
- board text added: "10K"
- board text added: "1838B"
- board text added: "22"
- board text added: "8"
- board text added: "A"
- board text added: "B"
- board text added: "C"
- board text added: "D"
- board text added: "GND"
- board text added: "IR LED"
- board text added: "IRis"
- board text added: "Red LED"
- board text added: "Vcc"
