File: Circuit/IRis - Slave Schematic.sch (EAGLE design)
At the start: 15 parts, among them U1 ATTINY85SU

Commit message: PCB Layout Added
Parts:
- R6: value 1k -> 22
- R7: value 33 -> 10k
Connections:
- removed net N$6: D1.C, D2.GND, LED1.C, R4.1, R5.1, U1.GND
- new net N$10: D2.VCC, R1.2, R5.2, U1.PB0, U1.VCC
- new net N$12: R1.1, R2.2, S1.2
- net N$1: now also R2.1, R3.2; no longer R1.1, R2.2
- net N$2: now also R3.1, R4.2; no longer R2.1, R3.2
- net N$3: now also D1.C, LED1.C, R4.1; no longer R3.1, R4.2
- net N$4: now also D2.GND, U1.GND; no longer D2.VCC, R1.2, S1.2, U1.PB0, U1.VCC
- net N$5: now also R5.1; no longer R5.2
Other:
- moved on the sheet: D2, R5, S1, S2, S3, S4

Commit message: PCB Layout Included For AA Cell and CR2032 Cell. Gerber Files Added
Parts:
- renumbered D1 to RED_LED, D2 to VS1838B, LED1 to IR_LED
Connections:
- removed net N$4: U1.GND, VS1838B.GND
- net N$3: now also U1.GND, VS1838B.GND
Other:
- moved on the sheet: R7
Changed lines of the file:
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@@
 <part name="S4" library="SparkFun-Switches" deviceset="MOMENTARY-SWITCH-SPST" device="-PTH-6.0MM"/>
 <part name="U1" library="ATtiny85" deviceset="ATTINY85" device="SU"/>
-<part name="D1" library="led" library_urn="urn:adsk.eagle:library:259" deviceset="SFH482" device="" package3d_urn="urn:adsk.eagle:package:15795/1"/>
-<part name="D2" library="SparkFun-Sensors" deviceset="BRM-2508" device="RA"/>
-<part name="LED1" library="led" library_urn="urn:adsk.eagle:library:259" deviceset="TLLR4400" device="" package3d_urn="urn:adsk.eagle:package:15797/1"/>
+<part name="RED_LED" library="led" library_urn="urn:adsk.eagle:library:259" deviceset="SFH482" device="" package3d_urn="urn:adsk.eagle:package:15795/1"/>
+<part name="VS1838B" library="SparkFun-Sensors" deviceset="BRM-2508" device="RA"/>
+<part name="IR_LED" library="led" library_urn="urn:adsk.eagle:library:259" deviceset="TLLR4400" device="" package3d_urn="urn:adsk.eagle:package:15797/1"/>
 <part name="R6" library="SparkFun-Resistors" library_urn="urn:adsk.eagle:library:532" deviceset="1KOHM" device="-HORIZ-1/4W-5%" package3d_urn="urn:adsk.eagle:package:39658/1" value="22"/>
 <part name="R7" library="SparkFun-Resistors" library_urn="urn:adsk.eagle:library:532" deviceset="33OHM" device="-0603-1/10W-1%" package3d_urn="urn:adsk.eagle:package:39650/1" value="10k"/>
@@
 <instance part="S4" gate="G$1" x="10.16" y="15.24"/>
 <instance part="U1" gate="G$1" x="66.04" y="38.1"/>
-<instance part="D1" gate="1" x="68.58" y="15.24" rot="MR90"/>
-<instance part="D2" gate="G$1" x="45.72" y="0" rot="R90"/>
-<instance part="LED1" gate="G$1" x="68.58" y="2.54" rot="R270"/>
+<instance part="RED_LED" gate="1" x="68.58" y="15.24" rot="MR90"/>
+<instance part="VS1838B" gate="G$1" x="45.72" y="0" rot="R90"/>
+<instance part="IR_LED" gate="G$1" x="68.58" y="2.54" rot="R270"/>
 <instance part="R6" gate="G$1" x="78.74" y="2.54"/>
-<instance part="R7" gate="G$1" x="76.2" y="15.24"/>
+<instance part="R7" gate="G$1" x="78.74" y="15.24"/>
 <instance part="R1" gate="G$1" x="38.1" y="50.8" rot="R90"/>
 <instance part="R2" gate="G$1" x="38.1" y="40.64" rot="R90"/>
@@
 <wire x1="15.24" y1="15.24" x2="38.1" y2="15.24" width="0.1524" layer="91"/>
 <pinref part="R4" gate="G$1" pin="1"/>
-<pinref part="D1" gate="1" pin="C"/>
-<wire x1="38.1" y1="15.24" x2="60.96" y2="15.24" width="0.1524" layer="91"/>
-<pinref part="LED1" gate="G$1" pin="C"/>
+<pinref part="RED_LED" gate="1" pin="C"/>
+<wire x1="38.1" y1="15.24" x2="45.72" y2="15.24" width="0.1524" layer="91"/>
+<pinref part="IR_LED" gate="G$1" pin="C"/>
+<wire x1="45.72" y1="15.24" x2="60.96" y2="15.24" width="0.1524" layer="91"/>
 <wire x1="60.96" y1="15.24" x2="63.5" y2="15.24" width="0.1524" layer="91"/>
 <wire x1="63.5" y1="2.54" x2="60.96" y2="2.54" width="0.1524" layer="91"/>
@@
 <junction x="60.96" y="15.24"/>
 <junction x="38.1" y="15.24"/>
+<pinref part="U1" gate="G$1" pin="GND"/>
+<pinref part="VS1838B" gate="G$1" pin="GND"/>
+<wire x1="45.72" y1="7.62" x2="45.72" y2="15.24" width="0.1524" layer="91"/>
+<wire x1="45.72" y1="15.24" x2="45.72" y2="30.48" width="0.1524" layer="91"/>
+<wire x1="45.72" y1="30.48" x2="50.8" y2="30.48" width="0.1524" layer="91"/>
+<junction x="45.72" y="15.24"/>
 </segment>
 </net>
@@
 <wire x1="83.82" y1="40.64" x2="86.36" y2="40.64" width="0.1524" layer="91"/>
 <wire x1="86.36" y1="40.64" x2="86.36" y2="15.24" width="0.1524" layer="91"/>
-<wire x1="86.36" y1="15.24" x2="81.28" y2="15.24" width="0.1524" layer="91"/>
+<wire x1="86.36" y1="15.24" x2="83.82" y2="15.24" width="0.1524" layer="91"/>
 <pinref part="R7" gate="G$1" pin="2"/>
 </segment>
@@
 <pinref part="U1" gate="G$1" pin="PB2"/>
 <wire x1="91.44" y1="35.56" x2="83.82" y2="35.56" width="0.1524" layer="91"/>
-<pinref part="D2" gate="G$1" pin="OUT"/>
+<pinref part="VS1838B" gate="G$1" pin="OUT"/>
 <wire x1="91.44" y1="10.16" x2="43.18" y2="10.16" width="0.1524" layer="91"/>
 <wire x1="43.18" y1="10.16" x2="43.18" y2="7.62" width="0.1524" layer="91"/>
@@
 <segment>
 <pinref part="R6" gate="G$1" pin="1"/>
-<pinref part="LED1" gate="G$1" pin="A"/>
+<pinref part="IR_LED" gate="G$1" pin="A"/>
 <wire x1="73.66" y1="2.54" x2="71.12" y2="2.54" width="0.1524" layer="91"/>
 </segment>
@@
 <net name="N$9" class="0">
 <segment>
-<pinref part="D1" gate="1" pin="A"/>
+<pinref part="RED_LED" gate="1" pin="A"/>
 <pinref part="R7" gate="G$1" pin="1"/>
+<wire x1="73.66" y1="15.24" x2="71.12" y2="15.24" width="0.1524" layer="91"/>
 </segment>
 </net>
@@
 </segment>
 </net>
-<net name="N$4" class="0">
-<segment>
-<pinref part="U1" gate="G$1" pin="GND"/>
-<pinref part="D2" gate="G$1" pin="GND"/>
-<wire x1="45.72" y1="7.62" x2="45.72" y2="30.48" width="0.1524" layer="91"/>
-<wire x1="45.72" y1="30.48" x2="50.8" y2="30.48" width="0.1524" layer="91"/>
-</segment>
-</net>
 <net name="N$10" class="0">
 <segment>
@@
 <wire x1="83.82" y1="30.48" x2="96.52" y2="30.48" width="0.1524" layer="91"/>
 <wire x1="96.52" y1="30.48" x2="96.52" y2="55.88" width="0.1524" layer="91"/>
-<pinref part="D2" gate="G$1" pin="VCC"/>
+<pinref part="VS1838B" gate="G$1" pin="VCC"/>
 <pinref part="U1" gate="G$1" pin="VCC"/>
 <wire x1="48.26" y1="7.62" x2="48.26" y2="43.18" width="0.1524" layer="91"/>
